File: PCB/switch_connector/switch.brd (EAGLE design)
At the start: 40.3 x 44.4 mm, 7 parts

Commit message: all files
Parts:
- removed JP1: (no value), pinhead:2X03
- removed RF: (no value), pinhead:1X01
- added PAD1, PAD2, PAD3, PAD4, PAD5, PAD6, PAD7, PAD8, PAD9: WIREPADSMD5-2,5, wirepad:5-2,5
Connections:
- net GND: now also PAD5.1, PAD9.1; no longer JP1.3
- net N$1: now also PAD3.1; no longer JP1.2
- net N$10: now also PAD6.1; no longer JP1.5
- net N$2: now also PAD2.1; no longer JP1.4
- net N$3: now also PAD1.1; no longer JP1.6
- net N$7: now also PAD7.1; no longer RF.1
- net VCC: now also PAD4.1, PAD8.1; no longer JP1.1
Routing:
- net N$5: track 88.9 -> 0.00 mm
- net N$1: track 38.9 -> 14.5 mm, vias 1 -> 0
- net N$10: track 38.1 -> 14.1 mm, vias 1 -> 0
- net N$2: track 36.5 -> 14.9 mm, vias 1 -> 0
- net N$3: track 34.9 -> 15.3 mm, vias 1 -> 0
- net GND: track 41.4 -> 24.3 mm, vias 1 -> 0
- net N$7: track 10.7 -> 15.5 mm, vias 1 -> 0
- net VCC: track 13.8 -> 14.6 mm
- removed copper zone on layer 1, net GND
- removed copper zone on layer 1, net N$4
- removed copper zone on layer 16, net VCC
Other:
- board text removed: "+"
- board text removed: "-"

Commit message: Last changes
Parts:
- moved PAD8 6.48 mm to (7.62, 30.5), turned to 90 degrees
- moved PAD9 4.58 mm to (16.5, 34.3), turned to 90 degrees
Routing:
- net GND: track 24.3 -> 19.9 mm
- net VCC: track 14.6 -> 11.4 mm
Other:
- board text added: "GND"
- board text added: "VCC"
Changed lines of the file:
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@@
 <layer number="17" name="Pads" color="2" fill="1" visible="yes" active="yes"/>
 <layer number="18" name="Vias" color="2" fill="1" visible="yes" active="yes"/>
-<layer number="19" name="Unrouted" color="6" fill="1" visible="yes" active="yes"/>
+<layer number="19" name="Unrouted" color="6" fill="1" visible="no" active="yes"/>
 <layer number="20" name="Dimension" color="24" fill="1" visible="yes" active="yes"/>
-<layer number="21" name="tPlace" color="7" fill="1" visible="yes" active="yes"/>
-<layer number="22" name="bPlace" color="7" fill="1" visible="yes" active="yes"/>
-<layer number="23" name="tOrigins" color="15" fill="1" visible="yes" active="yes"/>
-<layer number="24" name="bOrigins" color="15" fill="1" visible="yes" active="yes"/>
-<layer number="25" name="tNames" color="7" fill="1" visible="yes" active="yes"/>
-<layer number="26" name="bNames" color="7" fill="1" visible="yes" active="yes"/>
-<layer number="27" name="tValues" color="7" fill="1" visible="yes" active="yes"/>
-<layer number="28" name="bValues" color="7" fill="1" visible="yes" active="yes"/>
-<layer number="29" name="tStop" color="7" fill="3" visible="yes" active="yes"/>
-<layer number="30" name="bStop" color="7" fill="6" visible="yes" active="yes"/>
-<layer number="31" name="tCream" color="7" fill="4" visible="yes" active="yes"/>
-<layer number="32" name="bCream" color="7" fill="5" visible="yes" active="yes"/>
-<layer number="33" name="tFinish" color="6" fill="3" visible="yes" active="yes"/>
-<layer number="34" name="bFinish" color="6" fill="6" visible="yes" active="yes"/>
-<layer number="35" name="tGlue" color="7" fill="4" visible="yes" active="yes"/>
-<layer number="36" name="bGlue" color="7" fill="5" visible="yes" active="yes"/>
-<layer number="37" name="tTest" color="7" fill="1" visible="yes" active="yes"/>
-<layer number="38" name="bTest" color="7" fill="1" visible="yes" active="yes"/>
-<layer number="39" name="tKeepout" color="4" fill="11" visible="yes" active="yes"/>
-<layer number="40" name="bKeepout" color="1" fill="11" visible="yes" active="yes"/>
-<layer number="41" name="tRestrict" color="4" fill="10" visible="yes" active="yes"/>
-<layer number="42" name="bRestrict" color="1" fill="10" visible="yes" active="yes"/>
-<layer number="43" name="vRestrict" color="2" fill="10" visible="yes" active="yes"/>
-<layer number="44" name="Drills" color="7" fill="1" visible="yes" active="yes"/>
-<layer number="45" name="Holes" color="7" fill="1" visible="yes" active="yes"/>
-<layer number="46" name="Milling" color="3" fill="1" visible="yes" active="yes"/>
-<layer number="47" name="Measures" color="7" fill="1" visible="yes" active="yes"/>
-<layer number="48" name="Document" color="7" fill="1" visible="yes" active="yes"/>
-<layer number="49" name="Reference" color="7" fill="1" visible="yes" active="yes"/>
-<layer number="51" name="tDocu" color="7" fill="1" visible="yes" active="yes"/>
-<layer number="52" name="bDocu" color="7" fill="1" visible="yes" active="yes"/>
+<layer number="21" name="tPlace" color="7" fill="1" visible="no" active="yes"/>
+<layer number="22" name="bPlace" color="7" fill="1" visible="no" active="yes"/>
+<layer number="23" name="tOrigins" color="15" fill="1" visible="no" active="yes"/>
+<layer number="24" name="bOrigins" color="15" fill="1" visible="no" active="yes"/>
+<layer number="25" name="tNames" color="7" fill="1" visible="no" active="yes"/>
+<layer number="26" name="bNames" color="7" fill="1" visible="no" active="yes"/>
+<layer number="27" name="tValues" color="7" fill="1" visible="no" active="yes"/>
+<layer number="28" name="bValues" color="7" fill="1" visible="no" active="yes"/>
+<layer number="29" name="tStop" color="7" fill="3" visible="no" active="yes"/>
+<layer number="30" name="bStop" color="7" fill="6" visible="no" active="yes"/>
+<layer number="31" name="tCream" color="7" fill="4" visible="no" active="yes"/>
+<layer number="32" name="bCream" color="7" fill="5" visible="no" active="yes"/>
+<layer number="33" name="tFinish" color="6" fill="3" visible="no" active="yes"/>
+<layer number="34" name="bFinish" color="6" fill="6" visible="no" active="yes"/>
+<layer number="35" name="tGlue" color="7" fill="4" visible="no" active="yes"/>
+<layer number="36" name="bGlue" color="7" fill="5" visible="no" active="yes"/>
+<layer number="37" name="tTest" color="7" fill="1" visible="no" active="yes"/>
+<layer number="38" name="bTest" color="7" fill="1" visible="no" active="yes"/>
+<layer number="39" name="tKeepout" color="4" fill="11" visible="no" active="yes"/>
+<layer number="40" name="bKeepout" color="1" fill="11" visible="no" active="yes"/>
+<layer number="41" name="tRestrict" color="4" fill="10" visible="no" active="yes"/>
+<layer number="42" name="bRestrict" color="1" fill="10" visible="no" active="yes"/>
+<layer number="43" name="vRestrict" color="2" fill="10" visible="no" active="yes"/>
+<layer number="44" name="Drills" color="7" fill="1" visible="no" active="yes"/>
+<layer number="45" name="Holes" color="7" fill="1" visible="no" active="yes"/>
+<layer number="46" name="Milling" color="3" fill="1" visible="no" active="yes"/>
+<layer number="47" name="Measures" color="7" fill="1" visible="no" active="yes"/>
+<layer number="48" name="Document" color="7" fill="1" visible="no" active="yes"/>
+<layer number="49" name="Reference" color="7" fill="1" visible="no" active="yes"/>
+<layer number="51" name="tDocu" color="7" fill="1" visible="no" active="yes"/>
+<layer number="52" name="bDocu" color="7" fill="1" visible="no" active="yes"/>
 <layer number="88" name="SimResults" color="9" fill="1" visible="no" active="no"/>
 <layer number="89" name="SimProbes" color="9" fill="1" visible="no" active="no"/>
@@
 <circle x="35.687" y="5.08" radius="1.27" width="0.1524" layer="1"/>
 <circle x="20.828" y="40.894" radius="1.27" width="0.1524" layer="1"/>
+<text x="7.62" y="34.29" size="0.8128" layer="16" rot="MR180">VCC</text>
+<text x="17.78" y="36.83" size="0.8128" layer="16" rot="MR0">GND</text>
 </plain>
 <attributes>
@@
 <element name="PAD6" library="wirepad" library_urn="urn:adsk.eagle:library:412" package="5-2,5" package3d_urn="urn:adsk.eagle:package:30845/1" value="WIREPADSMD5-2,5" x="29.337" y="26.162"/>
 <element name="PAD7" library="wirepad" library_urn="urn:adsk.eagle:library:412" package="5-2,5" package3d_urn="urn:adsk.eagle:package:30845/1" value="WIREPADSMD5-2,5" x="6.35" y="17.78"/>
-<element name="PAD8" library="wirepad" library_urn="urn:adsk.eagle:library:412" package="5-2,5" package3d_urn="urn:adsk.eagle:package:30845/1" value="WIREPADSMD5-2,5" x="6.35" y="36.83"/>
-<element name="PAD9" library="wirepad" library_urn="urn:adsk.eagle:library:412" package="5-2,5" package3d_urn="urn:adsk.eagle:package:30845/1" value="WIREPADSMD5-2,5" x="12.7" y="36.83"/>
+<element name="PAD8" library="wirepad" library_urn="urn:adsk.eagle:library:412" package="5-2,5" package3d_urn="urn:adsk.eagle:package:30845/1" value="WIREPADSMD5-2,5" x="7.62" y="30.48" rot="R90"/>
+<element name="PAD9" library="wirepad" library_urn="urn:adsk.eagle:library:412" package="5-2,5" package3d_urn="urn:adsk.eagle:package:30845/1" value="WIREPADSMD5-2,5" x="16.51" y="34.29" rot="R90"/>
 </elements>
 <signals>
@@
 <wire x1="22.098" y1="27.432" x2="22.098" y2="30.988" width="2.54" layer="1"/>
 <contactref element="PAD9" pad="1"/>
-<wire x1="12.7" y1="36.83" x2="22.098" y2="27.432" width="2.54" layer="1"/>
+<wire x1="16.51" y1="34.29" x2="22.098" y2="27.432" width="2.54" layer="1"/>
 <wire x1="22.098" y1="27.432" x2="22.098" y2="26.416" width="2.54" layer="1"/>
 <wire x1="22.098" y1="26.416" x2="22.098" y2="25.908" width="0" layer="19" extent="1-1"/>
@@
 <contactref element="PAD4" pad="1"/>
 <contactref element="PAD8" pad="1"/>
-<wire x1="6.35" y1="36.83" x2="6.35" y2="33.02" width="2.54" layer="1"/>
-<wire x1="6.35" y1="33.02" x2="13.97" y2="25.4" width="2.54" layer="1"/>
+<wire x1="7.62" y1="30.48" x2="7.62" y2="25.4" width="2.54" layer="1"/>
+<wire x1="7.62" y1="25.4" x2="13.97" y2="25.4" width="2.54" layer="1"/>
 <wire x1="13.97" y1="25.4" x2="13.97" y2="25.781" width="0" layer="19" extent="1-1"/>
 </signal>
