File: PCB/EhomeLightController/ehomeLight_doit.brd (EAGLE design)
At the start: 89.8 x 83.8 mm, 8 parts

Commit message: all files
Parts:
- removed IN1-1, IN1-2: (no value), con-wago-508:W237-7P
- added X10, X11, X12, X13, X6, X7, X8, X9: (no value), con-wago-500:W237-102
- added X3: (no value), con-wago-508:W237-132
- X1: device con-wago-508:W237-6P -> con-wago-500:W237-102
- moved X1 10.0 mm to (83.7, 78.2)
- moved X5 8.64 mm to (40.3, 5.08)
Connections:
- removed net GPIO0: SV1.14, X4.2
- removed net GPIO23: IN1-1.7, SV1.2
- new net GPIO12: SV2.12
- new net GPIO13: X7.2
- new net GPIO14: SV2.11
- new net GPIO2: SV1.12, X4.2
- new net N$1: X7.1
- new net N$2: SV2.13
- new net N$3: SV1.1, X10.1
- net GND: now also SV2.17; no longer SV2.14
- net GPIO15: now also SV1.13; no longer SV1.16
- net GPIO16: now also SV1.10; no longer SV1.12
- net GPIO17: now also SV1.9, X6.1; no longer IN1-1.1, SV1.11
- net GPIO18: now also SV1.7, X8.1; no longer IN1-1.3, SV1.9
- net GPIO19: now also SV1.6, X8.2; no longer IN1-1.4, SV1.8
- net GPIO21: now also SV1.5, X9.1; no longer IN1-1.5, SV1.6
- net GPIO22: now also SV1.2, X9.2; no longer IN1-1.6, SV1.3
- net GPIO25: now also SV2.8, X10.2; no longer IN1-2.1, SV2.9
- net GPIO26: now also SV2.9; no longer SV2.10
- net GPIO27: now also SV2.10; no longer SV2.11
- net GPIO32: now also SV2.6, X13.2; no longer IN1-2.3, SV2.7
- net GPIO33: now also SV2.7, X13.1; no longer IN1-2.2, SV2.8
- net GPIO34: now also SV2.4, X12.2; no longer IN1-2.5, SV2.5
- net GPIO35: now also SV2.5, X12.1; no longer IN1-2.4, SV2.6
- net GPIO36: now also SV2.2, X11.2; no longer IN1-2.7, SV2.3
- net GPIO39: now also SV2.3, X11.1; no longer IN1-2.6, SV2.4
- net GPIO4: now also SV1.11; no longer SV1.13
- net GPIO5: now also SV1.8, X6.2; no longer IN1-1.2, SV1.10
- net PWR: now also SV2.18; no longer SV2.19
Routing:
- net GPIO2: track 0.00 -> 55.7 mm
- net GND: track 145.7 -> 91.2 mm
- net GPIO0: track 53.7 -> 0.00 mm
- net N$3: track 0.00 -> 49.4 mm
- net GPIO23: track 40.2 -> 0.00 mm
- net GPIO19: track 66.7 -> 49.9 mm
- net GPIO18: track 72.1 -> 57.5 mm
- net GPIO5: track 74.4 -> 62.2 mm
- net GPIO21: track 55.5 -> 43.8 mm
- net GPIO17: track 78.9 -> 68.2 mm
- net PWR: track 111.2 -> 121.7 mm
- net GPIO22: track 42.8 -> 36.3 mm
- net GPIO27: track 63.1 -> 67.6 mm
- net GPIO26: track 57.7 -> 62.1 mm
- net GPIO4: track 47.2 -> 50.3 mm
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- added copper zone on layer 16, net GND

Commit message: Last changes
Connections:
- net N$3 renamed GPIO23
- removed net GPIO16: SV1.10, X4.4
- removed net GPIO2: SV1.12, X4.2
- removed net GPIO4: SV1.11, X4.3
Routing:
- net GPIO17: track 68.2 -> 0.00 mm
- net GPIO5: track 62.2 -> 0.00 mm
- net GPIO18: track 57.5 -> 0.00 mm
- net GPIO2: track 55.7 -> 0.00 mm
- net GPIO4: track 50.3 -> 0.00 mm
- net GPIO16: track 42.0 -> 0.00 mm
Other:
- board text added: "Light Controller doit v1"
Changed lines of the file:
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@@
 <grid distance="50" unitdist="mil" unit="mm" style="lines" multiple="1" display="yes" altdistance="5" altunitdist="mil" altunit="mil"/>
 <layers>
-<layer number="1" name="Top" color="4" fill="1" visible="no" active="yes"/>
+<layer number="1" name="Top" color="4" fill="1" visible="yes" active="yes"/>
 <layer number="16" name="Bottom" color="1" fill="1" visible="yes" active="yes"/>
 <layer number="17" name="Pads" color="2" fill="1" visible="yes" active="yes"/>
@@
 <wire x1="89.84" y1="83.81" x2="0" y2="83.81" width="0.2" layer="20"/>
 <wire x1="0" y1="83.81" x2="0" y2="0" width="0.2" layer="20"/>
-<rectangle x1="0.127" y1="28.702" x2="57.127" y2="83.702" layer="1"/>
 <hole x="2.413" y="81.407" drill="4"/>
 <hole x="54.229" y="81.534" drill="4"/>
 <hole x="2.286" y="30.861" drill="4"/>
 <hole x="54.737" y="30.988" drill="4"/>
+<text x="40.259" y="80.391" size="1.778" layer="16" rot="MR0">Light Controller doit v1</text>
 </plain>
 <attributes>
@@
 <wire x1="35.56" y1="49.53" x2="15.24" y2="29.21" width="1.016" layer="16"/>
 </signal>
-<signal name="GPIO4">
-<contactref element="X4" pad="3"/>
-<contactref element="SV1" pad="11"/>
-<wire x1="60.96" y1="44.45" x2="38.1" y2="44.45" width="1.016" layer="16"/>
-<wire x1="38.1" y1="44.45" x2="25.4" y2="31.75" width="1.016" layer="16"/>
-<wire x1="25.4" y1="31.75" x2="25.4" y2="22.225" width="1.016" layer="16"/>
-</signal>
 <signal name="GPIO25">
 <contactref element="SV2" pad="8"/>
@@
 <contactref element="SV1" pad="9"/>
 <contactref element="X6" pad="1"/>
-<wire x1="51.25" y1="39.25" x2="60.75" y2="39.25" width="1" layer="16"/>
-<wire x1="25" y1="13" x2="51.25" y2="39.25" width="1" layer="16"/>
-<wire x1="15.75" y1="13" x2="25" y2="13" width="1" layer="16"/>
-<wire x1="7.25" y1="4.5" x2="15.75" y2="13" width="1" layer="16"/>
-<wire x1="60.75" y1="39.25" x2="60.96" y2="39.37" width="1" layer="16"/>
-<wire x1="7.25" y1="4.5" x2="7.152" y2="4.445" width="1" layer="16"/>
+<wire x1="7.152" y1="4.445" x2="60.96" y2="39.37" width="0" layer="19" extent="1-1"/>
 </signal>
 <signal name="GPIO5">
 <contactref element="SV1" pad="8"/>
 <contactref element="X6" pad="2"/>
-<wire x1="51.5" y1="36.75" x2="60.75" y2="36.75" width="1" layer="16"/>
-<wire x1="25.75" y1="11" x2="51.5" y2="36.75" width="1" layer="16"/>
-<wire x1="18.75" y1="11" x2="25.75" y2="11" width="1" layer="16"/>
-<wire x1="12.25" y1="4.5" x2="18.75" y2="11" width="1" layer="16"/>
-<wire x1="60.75" y1="36.75" x2="60.96" y2="36.83" width="1" layer="16"/>
-<wire x1="12.25" y1="4.5" x2="12.152" y2="4.445" width="1" layer="16"/>
+<wire x1="12.152" y1="4.445" x2="60.96" y2="36.83" width="0" layer="19" extent="1-1"/>
 </signal>
 <signal name="GPIO18">
 <contactref element="SV1" pad="7"/>
 <contactref element="X8" pad="1"/>
-<wire x1="60" y1="34.25" x2="60.75" y2="34.25" width="1" layer="16"/>
-<wire x1="59.5" y1="35.02" x2="60" y2="34.25" width="1" layer="16"/>
-<wire x1="52.23" y1="35.02" x2="59.5" y2="35.02" width="1" layer="16"/>
-<wire x1="43.98" y1="26.77" x2="52.23" y2="35.02" width="1" layer="16"/>
-<wire x1="44" y1="25.5" x2="43.98" y2="26.77" width="1" layer="16"/>
-<wire x1="27.5" y1="9" x2="44" y2="25.5" width="1" layer="16"/>
-<wire x1="25.5" y1="9" x2="27.5" y2="9" width="1" layer="16"/>
-<wire x1="23.5" y1="7" x2="25.5" y2="9" width="1" layer="16"/>
-<wire x1="21.25" y1="7" x2="23.5" y2="7" width="1" layer="16"/>
-<wire x1="18.75" y1="4.5" x2="21.25" y2="7" width="1" layer="16"/>
-<wire x1="17.5" y1="4.5" x2="18.75" y2="4.5" width="1" layer="16"/>
-<wire x1="60.75" y1="34.25" x2="60.96" y2="34.29" width="1" layer="16"/>
-<wire x1="17.5" y1="4.5" x2="17.312" y2="4.445" width="1" layer="16"/>
+<wire x1="17.312" y1="4.445" x2="60.96" y2="34.29" width="0" layer="19" extent="1-1"/>
 </signal>
 <signal name="GPIO19">
@@
 <wire x1="22.5" y1="4.5" x2="22.312" y2="4.445" width="1" layer="16"/>
 </signal>
-<signal name="GPIO2">
-<contactref element="X4" pad="2"/>
-<contactref element="SV1" pad="12"/>
-<wire x1="60.96" y1="46.99" x2="36.83" y2="46.99" width="1.016" layer="16"/>
-<wire x1="36.83" y1="46.99" x2="20.32" y2="30.48" width="1.016" layer="16"/>
-<wire x1="20.32" y1="30.48" x2="20.32" y2="22.225" width="1.016" layer="16"/>
-</signal>
-<signal name="GPIO16">
-<contactref element="X4" pad="4"/>
-<contactref element="SV1" pad="10"/>
-<wire x1="60.96" y1="41.91" x2="44.45" y2="41.91" width="1.016" layer="16"/>
-<wire x1="44.45" y1="41.91" x2="30.48" y2="27.94" width="1.016" layer="16"/>
-<wire x1="30.48" y1="27.94" x2="30.48" y2="22.225" width="1.016" layer="16"/>
-</signal>
 <signal name="GPIO26">
 <contactref element="X5" pad="2"/>
@@
 <contactref element="SV2" pad="13"/>
 </signal>
-<signal name="N$3">
+<signal name="GPIO23">
 <contactref element="SV1" pad="1"/>
 <contactref element="X10" pad="1"/>
