File: PCB/EhomeLightController/ehomeGeneral_v1.brd (EAGLE design)
At the start: 89.8 x 83.8 mm, 15 parts

Commit message: latest and greatest
Parts:
- added X14, X15: (no value), con-wago-500:W237-102
- X2: device con-wago-508:W237-132 -> con-wago-500:W237-102
- X4: device con-wago-508:W237-4P -> con-wago-500:W237-102
- moved X3 81.0 mm to (40.1, 5.08), turned to 0 degrees
- moved X10 78.6 mm to (19.9, 78.1), turned to 180 degrees
- moved X6 72.4 mm to (9.78, 78.1), turned to 180 degrees
- moved X4 55.7 mm to (30.0, 78.1), turned to 180 degrees
- moved X2 21.1 mm to (19.9, 5.71), flipped to the bottom
- moved X7 13.2 mm to (50.2, 78.1)
- moved X5 10.1 mm to (50.3, 5.08)
- moved X8 10.0 mm to (9.78, 5.71)
- moved X11 0.13 mm to (80.6, 5.71)
- moved X13 0.08 mm to (60.5, 5.71)
Connections:
- removed net N$1: X7.1
- removed net N$2: SV2.13
- removed net N$3: SV1.1, X10.1
- new net EN: SV2.1, X6.1
- new net GND1: SV1.3, X2.1
- new net GPIO0: SV1.14, X14.2
- new net GPIO23: SV1.1, X9.2
- new net PWR1: SV1.4, X2.2
- net GND: no longer X2.1
- net GPIO12: now also X15.1
- net GPIO13: now also SV2.13, X15.2; no longer X7.2
- net GPIO14: now also X3.1
- net GPIO15: now also X14.1; no longer X4.1
- net GPIO16: now also X10.1; no longer X4.4
- net GPIO17: now also X7.2; no longer X6.1
- net GPIO18: now also X6.2; no longer X8.1
- net GPIO19: now also X8.1; no longer X8.2
- net GPIO2: now also X4.1; no longer X4.2
- net GPIO21: now also X8.2; no longer X9.1
- net GPIO22: now also X9.1; no longer X9.2
- net GPIO25: now also X5.2; no longer X10.2
- net GPIO26: now also X5.1; no longer X5.2
- net GPIO27: now also X3.2; no longer X5.1
- net GPIO4: now also X4.2; no longer X4.3
- net GPIO5: now also X7.1; no longer X6.2
- net PWR: no longer X2.2
Routing:
- net PWR: track 121.7 -> 22.6 mm
- net GPIO14: track 0.00 -> 96.4 mm
- net GND: track 91.2 -> 23.4 mm
- net PWR1: track 0.00 -> 52.8 mm
- net N$3: track 49.4 -> 0.00 mm
- net GPIO12: track 0.00 -> 48.0 mm
- net GND1: track 0.00 -> 46.7 mm
- net GPIO13: track 0.00 -> 42.8 mm
- net GPIO0: track 0.00 -> 36.1 mm
- net GPIO5: track 62.2 -> 97.8 mm
- net GPIO23: track 0.00 -> 34.6 mm
- net GPIO18: track 57.5 -> 80.4 mm
- net GPIO15: track 61.1 -> 40.4 mm
- net GPIO21: track 43.8 -> 58.9 mm
- net GPIO19: track 49.9 -> 65.0 mm
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- removed copper zone on layer 16, net GND
Other:
- board text added: "Light Controller doit v2"
- board text removed: "Light Controller doit v1"
