File: PCB/EhomeLightController/ehomeLight_doit_v2.brd (EAGLE design)
At the start: 89.8 x 83.8 mm, 15 parts

Commit message: latest and greatest
Parts:
- moved X3 81.0 mm to (40.1, 5.08), turned to 0 degrees
- moved X10 73.7 mm to (63.4, 78.2), turned to 180 degrees
- moved X7 10.2 mm to (73.5, 78.2)
- moved X5 10.2 mm to (50.4, 5.08)
- moved X11 0.13 mm to (80.6, 5.75)
Connections:
- removed net GPIO2: SV1.12, X4.2
- removed net N$1: X7.1
- removed net N$2: SV2.13
- removed net N$3: SV1.1, X10.1
- new net EN: SV2.1
- new net GPIO23: SV1.1, X9.2
- net GPIO13: now also SV2.13; no longer X7.2
- net GPIO14: now also X3.1
- net GPIO16: now also X4.2; no longer X4.4
- net GPIO17: now also X4.3; no longer X6.1
- net GPIO18: now also X6.2; no longer X8.1
- net GPIO19: now also X8.1; no longer X8.2
- net GPIO21: now also X8.2; no longer X9.1
- net GPIO22: now also X9.1; no longer X9.2
- net GPIO25: now also X5.2; no longer X10.2
- net GPIO26: now also X5.1; no longer X5.2
- net GPIO27: now also X3.2; no longer X5.1
- net GPIO4: now also X6.1; no longer X4.3
- net GPIO5: now also X4.4; no longer X6.2
Routing:
- net GPIO14: track 0.00 -> 96.4 mm
- net GPIO2: track 55.7 -> 0.00 mm
- net N$3: track 49.4 -> 3.81 mm, vias 0 -> 1
- net GPIO23: track 0.00 -> 34.5 mm
- net GPIO4: track 50.3 -> 79.3 mm
- net GPIO5: track 62.2 -> 36.5 mm
- net GPIO17: track 68.2 -> 42.6 mm
- net GPIO16: track 42.0 -> 48.8 mm
- net GPIO25: track 51.7 -> 57.7 mm
- net GPIO33: track 45.9 -> 51.6 mm
- net GPIO32: track 40.1 -> 45.8 mm
- net GPIO35: track 34.7 -> 40.1 mm
- net GPIO21: track 43.8 -> 48.9 mm
- net GPIO36: track 24.0 -> 18.9 mm
- net GPIO19: track 49.9 -> 54.9 mm
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Other:
- board text added: "Light Controller doit v2"
- board text removed: "Light Controller doit v1"
