File: PCB/EhomeShades/ehomeShades_doit_v2.brd (EAGLE design)
At the start: 89.8 x 83.8 mm, 15 parts

Commit message: latest and greatest
Parts:
- removed X10, X11, X12, X7: (no value), con-wago-500:W237-102
- added SV3, SV4: (no value), con-lsta:FE20
- added X14, X15: (no value), con-wago-508:W237-132
- added X16, X17, X18, X19, X20, X21: (no value), con-wago-500:W237-102
- X2: device con-wago-508:W237-132 -> con-wago-500:W237-102
- moved X2 79.3 mm to (74.9, 64.8)
- moved X3 74.7 mm to (61.7, 5.08), turned to 0 degrees
- moved X5 31.8 mm to (72.0, 5.08)
- moved X6 22.9 mm to (32.5, 5.75)
- moved X8 22.9 mm to (42.7, 5.75)
- moved X9 21.6 mm to (51.6, 5.75)
- moved X13 20.3 mm to (80.9, 5.75)
- moved X4 18.5 mm to (17.8, 5.08)
Connections:
- removed net GPIO34: SV2.4, X12.2
- removed net GPIO35: SV2.5, X12.1
- removed net GPIO36: SV2.2, X11.2
- removed net GPIO39: SV2.3, X11.1
- removed net N$1: X7.1
- removed net N$2: SV2.13
- removed net N$3: SV1.1, X10.1
- new net EN: SV2.1, X2.1
- new net EN1: SV4.1, X2.2
- new net GPIO1: SV4.8, X14.2
- new net GPIO20: SV3.7, X16.2
- new net GPIO23: SV1.1, X9.2
- new net GPIO24: SV3.6, X17.1
- new net GPIO28: SV4.9, X14.1
- new net GPIO29: SV4.10, X15.2
- new net GPIO3: SV4.3, X19.1
- new net GPIO30: SV4.11, X15.1
- new net GPIO31: SV4.13
- new net GPIO40: SV3.5, X17.2
- new net GPIO41: SV3.2, X18.1
- new net GPIO42: SV3.1, X18.2
- new net GPIO43: SV3.11, X16.1
- new net GPIO44: SV4.12
- new net GPIO6: SV4.4, X20.2
- new net GPIO7: SV4.5, X20.1
- new net GPIO8: SV4.6, X21.2
- new net GPIO9: SV4.7, X21.1
- net GND: now also SV4.17; no longer X2.1
- net GPIO13: now also SV2.13; no longer X7.2
- net GPIO14: now also X3.1
- net GPIO16: now also X4.2; no longer X4.4
- net GPIO17: now also X4.3; no longer X6.1
- net GPIO18: now also X6.2; no longer X8.1
- net GPIO19: now also X8.1; no longer X8.2
- net GPIO2: now also SV4.2, X19.2; no longer SV1.12, X4.2
- net GPIO21: now also X8.2; no longer X9.1
- net GPIO22: now also X9.1; no longer X9.2
- net GPIO25: now also X5.2; no longer X10.2
- net GPIO26: now also X5.1; no longer X5.2
- net GPIO27: now also X3.2; no longer X5.1
- net GPIO4: now also X6.1; no longer X4.3
- net GPIO5: now also X4.4; no longer X6.2
- net PWR: now also SV4.18; no longer X2.2
Routing:
- net PWR: track 121.7 -> 0.00 mm
- net GPIO17: track 68.2 -> 0.00 mm
- net GND: track 91.2 -> 23.4 mm
- net GPIO27: track 67.6 -> 0.00 mm
- net GPIO5: track 62.2 -> 0.00 mm
- net GPIO26: track 62.1 -> 0.00 mm
- net GPIO15: track 61.1 -> 0.00 mm
- net GPIO18: track 57.5 -> 0.00 mm
- net GPIO2: track 55.7 -> 0.00 mm
- net GPIO25: track 51.7 -> 0.00 mm
- net GPIO4: track 50.3 -> 0.00 mm
- net GPIO19: track 49.9 -> 0.00 mm
- net N$3: track 49.4 -> 0.00 mm
- net GPIO33: track 45.9 -> 0.00 mm
- net GPIO21: track 43.8 -> 0.00 mm
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- removed copper zone on layer 16, net GND
Other:
- board text added: "Light Controller doit v2"
- board text removed: "Light Controller doit v1"
